Commit message: update xacro for gazebo and created launch file to get in running.

File: description/robot_model.xacro (robot description, xacro)
@@ -45,4 +45,7 @@
         </xacro:inertial_box>
     </link>
+    <gazebo reference="chasis">
+        <material>Gazebo/White</material>
+    </gazebo>
     <!-- LEFT WHEELS LINKS -->
     <joint name="base_to_left_wheel" type="continuous">
@@ -57,5 +60,5 @@
                 <cylinder radius="0.05" length="0.04"/>
             </geometry>
-            <material name="black"/>
+            <material name="blue"/>
         </visual>
         <collision>
@@ -68,4 +71,7 @@
         </xacro:inertial_cylinder>
     </link>
+    <gazebo reference="left_wheel">
+        <material>Gazebo/Blue</material>
+    </gazebo>
     <!-- RIGHT WHEELS LINKS -->
     <joint name="base_to_right_wheel" type="continuous">
@@ -80,5 +86,5 @@
                 <cylinder radius="0.05" length="0.04"/>
             </geometry>
-            <material name="black"/>
+            <material name="blue"/>
         </visual>
         <collision>
@@ -91,4 +97,7 @@
         </xacro:inertial_cylinder>
     </link>
+    <gazebo reference="right_wheel">
+        <material>Gazebo/Blue</material>
+    </gazebo>
     <!-- CASTOR WHEEL LINK -->
     <joint name="chasis_to_castor_wheel" type="fixed">
@@ -113,3 +122,6 @@
         </xacro:inertial_sphere>
     </link>
+    <gazebo reference="castor_wheel">
+        <material>Gazebo/Black</material>
+    </gazebo>
 </robot>
