Commit message: basic slam method added and code got more modular

File: description/robot.urdf.xacro (robot description, xacro)
@@ -1,5 +1,15 @@
 <?xml version="1.0"?>
 <robot xmlns:xacro="http://www.ros.org/wiki/xacro"  name="robot">
+    <xacro:arg name="use_ros2_control" default="true"/>
     <xacro:include filename="robot_model.xacro"/>
-    <xacro:include filename="gazebo_control.xacro"/>
+    <!--Conditional such that we can use either of ros2_control or gazebo_control-->
+    <xacro:if value="$(arg use_ros2_control)">
+        <xacro:include filename="ros2_control.xacro"/>
+    </xacro:if>
+    <xacro:unless value="$(arg use_ros2_control)">
+        <xacro:include filename="gazebo_control.xacro"/>
+    </xacro:unless>
+    <xacro:include filename="lidar.xacro"/>
+    <!-- <xacro:include filename="camera.xacro"/> We wouldn't want depth_camera and camera at the same time-->
+    <xacro:include filename="depth_camera.xacro"/>
 </robot>

File: description/robot_model.xacro (robot description, xacro)
@@ -21,4 +21,11 @@
     <!-- BASE LINK -->
     <link name="base_link"></link>
+    <!--BASE FOOTPRINT-->
+    <link name="base_footprint"/>
+    <joint name="base_footprint_joint" type="fixed">
+        <parent link="base_link"/>
+        <child link="base_footprint"/>
+        <origin xyz="0 0 0" ryp="0 0 0"/>
+    </joint>
     <!-- CHASIS LINK -->
     <joint name="base_to_chassis" type="fixed">
